File: Volterra IDEX Boards/Daughter Board/Daughter board.brd (EAGLE design)
At the start: 53 parts, among them J14 FEMALE 2x3, J5 455-1750-1-ND, J6 455-1750-1-ND, J7 455-1750-1-ND, K1 FFC/FPC/34PIN/1MMPITCH/TOPLOCK, X10 FIL_HEAT, X11 FIL_THM, X12 CH_THM, X13 CH_HEAT, X14 24V, X2 EXTDR-0, X3 EXTDR-1, X4 Z_LMT, X5 BED_THERM, X6 24V, X7 24V, X8 AUTO BED LEVELING, X9 Y_LMT

Commit message: Updated Daughter board schematic and other boards
Parts:
- removed HEADER: 455-1750-1-ND, SparkFun-Connectors:1X03
- removed J14: FEMALE 2x3, SparkFun-Connectors:2X3
- added J11, J8: (no value), SparkFun-Connectors:2X5_NOSILK
- added J12, J4: 455-1750-1-ND, SparkFun-Connectors:1X03
- added J13: (no value), SparkFun-Connectors:1X04
- added J15: (no value), SparkFun-Connectors:1X02
- added TP26: TEST-POINTTP_15TH_THRU, SparkFun-Connectors:TP_15TH
- added X15, X16: JST-XH-02-PIN-LONG-PAD, Rembrandt Electronics - JST XH Connectors v1-0:JST-XH-02-PACKAGE-LONG-PAD
- X1: device con-wago-500:W237-6 -> con-ptr500:AK500/4
- moved X1 134.7 mm to (44.5, -14.0)
- moved J5 114.6 mm to (48.3, 48.3)
- moved TP13 114.6 mm to (52.1, 36.8)
- moved TP17 114.6 mm to (62.2, 36.8)
- moved TP20 114.6 mm to (69.8, 36.8)
- moved TP6 114.6 mm to (34.3, 36.8)
- moved X10 114.6 mm to (69.8, 62.2)
- moved FRAME1 114.6 mm to (44.5, 78.7)
- moved J3 114.6 mm to (80.0, 40.6)
- moved J7 114.6 mm to (66.0, 48.3)
- moved TP10 114.6 mm to (44.5, 36.8)
- moved TP14 114.6 mm to (54.6, 36.8)
- moved TP18 114.6 mm to (64.8, 36.8)
- moved TP21 114.6 mm to (72.4, 36.8)
- moved TP24 114.6 mm to (80.0, 36.8)
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Connections:
- removed net N$10: J7.3
- removed net N$3: J5.3
- removed net N$6: J6.3
- removed net X_LMT: J5.1, K1.15, TP12.P$1
- new net 3V3: J4.3, J5.3, J6.3, J7.3
- new net X0_LMT: J4.1, K1.13, TP12.P$1, X16.1
- new net X1_LMT: J5.1, K1.12, TP26.P$1, X15.1
- net 24V: now also J12.1, K1.10; no longer K1.11, K1.12
- net 5V: now also J8.9; no longer J14.3, J14.4
- net A0+: now also J13.1
- net A0-: now also J13.2
- net A1+: now also J10.1
- net A1-: now also J10.2
- net B0+: now also J13.3
- net B0-: now also J13.4
- net B1+: now also J10.3
- net B1-: now also J10.4
- net CF+: now also J15.1, K1.24; no longer K1.26, X1.1
- net CF-: now also J15.2, K1.25; no longer K1.27, X1.2
- net GND: now also J12.2, J4.2, J8.10, K1.11, X15.2, X16.2; no longer J14.1, J14.2, K1.13, K1.14
- net H0+: now also K1.31, X1.2; no longer X1.3
- net H0-: now also X1.1; no longer K1.29, K1.30, K1.31, X1.4
- net H1+: now also K1.20, K1.21, K1.22, K1.27, K1.28, K1.29, K1.30, X1.4; no longer K1.24, K1.25, X1.5
- net H1-: now also K1.16, K1.17, K1.18, K1.19, X1.3; no longer K1.20, K1.21, K1.22, X1.6
- net PT0: now also J11.1, K1.26; no longer K1.28
- net PT1: now also J11.6, K1.15; no longer K1.19
- net SERVO_DAT: no longer J14.6, K1.16
- net Y_LMT: now also K1.14; no longer K1.18
- net Z_DIR: no longer J10.3, K1.17, X8.3
- net Z_OUT: now also J11.4, J12.3; no longer K1.10

Commit message: Added Daughter Board
Parts:
- removed J13: (no value), SparkFun-Connectors:1X04
- removed J8: (no value), SparkFun-Connectors:2X5_NOSILK
- removed J9: (no value), SparkFun-Connectors:2X5
- removed TP13, TP14, TP25: TEST-POINTTP_15TH_THRU, SparkFun-Connectors:TP_15TH
- removed X10: FIL_HEAT, Rembrandt Electronics - JST XH Connectors v1-0:JST-XH-02-PACKAGE-LONG-PAD
- removed X13: CH_HEAT, Rembrandt Electronics - JST XH Connectors v1-0:JST-XH-02-PACKAGE-LONG-PAD
- removed X14: 24V, Rembrandt Electronics - JST XH Connectors v1-0:JST-XH-02-PACKAGE-LONG-PAD
- removed X15, X16: JST-XH-02-PIN-LONG-PAD, Rembrandt Electronics - JST XH Connectors v1-0:JST-XH-02-PACKAGE-LONG-PAD
- J10: device SparkFun-Connectors:1X04 -> SparkFun-Connectors:1X02
- J12: value 455-1750-1-ND -> RGB LED
- X9: value Y_LMT -> RGB LED; device Rembrandt Electronics - JST XH Connectors v1-0:JST-XH-02-PACKAGE-LONG-PAD -> Rembrandt Electronics - JST XH Connectors v1-0:JST-XH-03-PACKAGE-LONG-PAD
- moved TP26 287.2 mm to (272.9, 124.5), flipped to the bottom, turned to 90 degrees
- moved TP9 258.9 mm to (273.0, 153.6), flipped to the bottom, turned to 90 degrees
- moved J11 248.8 mm to (263.9, 153.6), turned to 270 degrees
- moved TP10 241.9 mm to (272.8, 116.6), flipped to the bottom, turned to 90 degrees
- moved TP16 241.4 mm to (272.9, 150.0), flipped to the bottom, turned to 90 degrees
- moved TP2 241.3 mm to (234.0, 155.8), flipped to the bottom
- moved TP3 241.2 mm to (236.5, 155.7), flipped to the bottom
- moved TP4 241.1 mm to (238.9, 155.7), flipped to the bottom
- moved TP11 240.4 mm to (272.8, 119.3), flipped to the bottom, turned to 90 degrees
- moved J12 239.4 mm to (241.0, 107.9)
- moved TP12 238.8 mm to (272.7, 121.7), flipped to the bottom, turned to 90 degrees
- moved X12 236.3 mm to (251.3, 133.9), turned to 90 degrees
- moved J4 236.1 mm to (250.4, 104.6), turned to 90 degrees
- moved TP15 233.8 mm to (272.9, 126.9), flipped to the bottom, turned to 90 degrees
- moved TP19 231.6 mm to (272.8, 143.6), flipped to the bottom, turned to 270 degrees
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Connections:
- removed net CH_HEAT: J9.7, TP25.P$1, X13.1
- removed net FIL_HEAT: J9.8, X10.1
- removed net SERVO_DAT: TP13.P$1
- removed net Z_DIR: TP14.P$1
- new net PB0: J12.2, X9.2
- net 24V: now also J10.1, J10.2; no longer J12.1, X14.1
- net 5V: now also J12.3, X9.3; no longer J8.9
- net A0+: no longer J13.1
- net A0-: no longer J13.2
- net A1+: no longer J10.1
- net A1-: no longer J10.2
- net B0+: no longer J13.3
- net B0-: no longer J13.4
- net B1+: no longer J10.3
- net B1-: no longer J10.4
- net GND: now also J12.1, X9.1; no longer J12.2, J8.10, X10.2, X13.2, X14.2, X15.2, X16.2, X9.2
- net H0-: now also K1.27, K1.28, K1.29, K1.30
- net H1+: no longer K1.27, K1.28, K1.29, K1.30
- net PT0: no longer J9.2
- net PT1: no longer J9.4
- net X0_LMT: no longer X16.1
- net X1_LMT: no longer X15.1
- net Y_LMT: no longer X9.1
- net Z_OUT: now also J11.3; no longer J11.4, J12.3, J9.6
Routing:
- net GND: track 0.00 -> 193.8 mm
- net 24V: track 0.00 -> 180.9 mm, vias 0 -> 3
- net Y_LMT: track 0.00 -> 156.1 mm, vias 0 -> 2
- net 5V: track 0.00 -> 147.4 mm, vias 0 -> 4
- net H1+: track 0.00 -> 142.9 mm, vias 0 -> 3
- net H1-: track 0.00 -> 137.6 mm, vias 0 -> 3
- net CF-: track 0.00 -> 137.2 mm, vias 0 -> 1
- net CF+: track 0.00 -> 135.2 mm, vias 0 -> 2
- net H0-: track 0.00 -> 125.0 mm
- net X0_LMT: track 0.00 -> 124.4 mm, vias 0 -> 1
- net H0+: track 0.00 -> 124.3 mm
- net PT0: track 0.00 -> 120.6 mm, vias 0 -> 1
- net X1_LMT: track 0.00 -> 111.1 mm, vias 0 -> 2
- net PT1: track 0.00 -> 108.4 mm, vias 0 -> 2
- net Z_LMT: track 0.00 -> 76.3 mm
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- added copper zone on layer 1, net GND
- added copper zone on layer 16, net GND
Other:
- board outline added: 114.3 x 69.8 mm
- board text added: "24V"
- board text added: "5V"
- board text added: "@vjvarada"
- board text added: "A0+"
- board text added: "A0-"
- board text added: "A1+"
- board text added: "A1-"
- board text added: "B0+"
- board text added: "B0-"
- board text added: "B1+"
- board text added: "B1-"
- board text added: "CF+"
- board text added: "CF-"
- board text added: "Designed by"
- board text added: "GND"
- board text added: "H0+"
- board text added: "H0-"
- board text added: "H1+"
- board text added: "H1-"
- board text added: "PT0"
- board text added: "PT1"
- board text added: "Volterra IDEX Daughter Board BTT Octopus V1.0 V1.0"
- board text added: "X0_LMT"
- board text added: "X1_LMT"
- board text added: "Y_LMT"
- board text added: "Z_OUT"
