File: Volterra IDEX Boards/Carriage 1 board/Carriage Board 1.brd (EAGLE design)
At the start: 84.5 x 61.3 mm, 20 parts, among them K1 FFC/FPC/34PIN/1MMPITCH/TOPLOCK, K2 Tool 0, X1 EXTDR-0, X4 24V, X5 X_LMT

Commit message: Updated Daughter board schematic and other boards
Connections:
- net 5V: now also K2.3
Routing:
- net 5V: track 0.00 -> 65.5 mm
Changed lines of the file:
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@@
 <signal name="5V">
 <contactref element="K1" pad="22"/>
+<contactref element="K2" pad="3"/>
+<wire x1="58.443" y1="50.0302" x2="58.42" y2="50.0532" width="0.6096" layer="1"/>
+<wire x1="58.42" y1="50.0532" x2="58.42" y2="54.61" width="0.6096" layer="1"/>
+<wire x1="58.42" y1="54.61" x2="52.705" y2="60.325" width="0.6096" layer="1"/>
+<wire x1="29.845" y1="60.325" x2="27.94" y2="58.42" width="0.6096" layer="1"/>
+<wire x1="27.94" y1="58.42" x2="27.94" y2="41.275" width="0.6096" layer="1"/>
+<wire x1="33.875" y1="35.34" x2="35.628" y2="35.34" width="0.6096" layer="1"/>
+<wire x1="52.705" y1="60.325" x2="29.845" y2="60.325" width="0.6096" layer="1"/>
+<wire x1="27.94" y1="41.275" x2="33.875" y2="35.34" width="0.6096" layer="1"/>
 </signal>
 <signal name="PT1">

Commit message: Board files added
Parts:
- moved TP9 0.18 mm to (52.6, 31.6), flipped to the bottom
- flipped TP1 to the bottom
- flipped TP10 to the bottom
- flipped TP11 to the bottom
- flipped TP12 to the bottom
- flipped TP13 to the bottom
- flipped TP3 to the bottom
- flipped TP5 to the bottom
- flipped TP6 to the bottom
- flipped TP7 to the bottom
- flipped TP8 to the bottom
- flipped X4 to the top
- flipped X5 to the top
Routing:
- net GND: track 73.8 -> 78.8 mm, vias 0 -> 3
- net 24V: track 96.0 -> 100.7 mm, vias 0 -> 1
- net B1+: track 45.5 -> 45.9 mm, vias 2 -> 3
- net X1_LMT: track 44.9 -> 44.5 mm, vias 0 -> 1
- net H1+: track 47.4 -> 47.5 mm, vias 1 -> 2
- net H1-: vias 1 -> 2
- net CF+: vias 1 -> 2
- net A1-: vias 0 -> 1
- net CF-: vias 1 -> 2
- net B1-: vias 0 -> 1
- net A1+: vias 0 -> 1
