File: Volterra IDEX Boards/Chassis board/Chassis board.sch (EAGLE design)
At the start: 27 parts, among them K1 FFC/FPC/34PIN/1MMPITCH/TOPLOCK, K2 FFC/FPC/34PIN/1MMPITCH/TOPLOCK, K3 FFC/FPC/34PIN/1MMPITCH/TOPLOCK

Commit message: Switching of carriage board numbering, changing extruder FFC pins and fixing routings
Connections:
- removed net X2_LMT: K1.23, K3.17, TP12.1
- new net X0_LMT: K1.22, K2.18, TP5.1
- net X1_LMT: now also K1.23, K3.17, TP12.1; no longer K1.22, K2.18, TP5.1
Changed lines of the file:
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@@
-</segment>
-</net>
-<net name="X1_LMT" class="0">
-<segment>
-<pinref part="K1" gate="G$1" pin="22"/>
-<wire x1="114.3" y1="35.56" x2="114.3" y2="55.88" width="0.1524" layer="91"/>
-<label x="114.3" y="55.88" size="1.778" layer="95" rot="R90"/>
-</segment>
-<segment>
-<pinref part="K2" gate="G$1" pin="18"/>
-<wire x1="40.64" y1="111.76" x2="60.96" y2="111.76" width="0.1524" layer="91"/>
-<label x="60.96" y="111.76" size="1.778" layer="95"/>
-</segment>
-<segment>
-<pinref part="TP5" gate="G$1" pin="1"/>
-<wire x1="91.44" y1="119.38" x2="86.36" y2="119.38" width="0.1524" layer="91"/>
-<label x="86.36" y="119.38" size="1.778" layer="95" rot="R180"/>
-</segment>
-</net>
-<net name="X2_LMT" class="0">
-<segment>
-<pinref part="K1" gate="G$1" pin="23"/>
-<wire x1="116.84" y1="35.56" x2="116.84" y2="55.88" width="0.1524" layer="91"/>
-<label x="116.84" y="55.88" size="1.778" layer="95" rot="R90"/>
-</segment>
-<segment>
-<pinref part="K3" gate="G$1" pin="17"/>
-<wire x1="210.82" y1="114.3" x2="190.5" y2="114.3" width="0.1524" layer="91"/>
-<label x="190.5" y="114.3" size="1.778" layer="95" rot="R180"/>
-</segment>
-<segment>
-<pinref part="TP12" gate="G$1" pin="1"/>
-<wire x1="137.16" y1="139.7" x2="134.62" y2="139.7" width="0.1524" layer="91"/>
-<label x="134.62" y="139.7" size="1.778" layer="95" rot="R180"/>
 </segment>
 </net>
@@
 </segment>
 </net>
+<net name="X0_LMT" class="0">
+<segment>
+<pinref part="K2" gate="G$1" pin="18"/>
+<wire x1="40.64" y1="111.76" x2="60.96" y2="111.76" width="0.1524" layer="91"/>
+<label x="60.96" y="111.76" size="1.778" layer="95"/>
+</segment>
+<segment>
+<pinref part="TP5" gate="G$1" pin="1"/>
+<wire x1="91.44" y1="119.38" x2="86.36" y2="119.38" width="0.1524" layer="91"/>
+<label x="86.36" y="119.38" size="1.778" layer="95" rot="R180"/>
+</segment>
+<segment>
+<pinref part="K1" gate="G$1" pin="22"/>
+<wire x1="114.3" y1="35.56" x2="114.3" y2="55.88" width="0.1524" layer="91"/>
+<label x="114.3" y="55.88" size="1.778" layer="95" rot="R90"/>
+</segment>
+</net>
+<net name="X1_LMT" class="0">
+<segment>
+<pinref part="K1" gate="G$1" pin="23"/>
+<wire x1="116.84" y1="35.56" x2="116.84" y2="55.88" width="0.1524" layer="91"/>
+<label x="116.84" y="55.88" size="1.778" layer="95" rot="R90"/>
+</segment>
+<segment>
+<pinref part="K3" gate="G$1" pin="17"/>
+<wire x1="210.82" y1="114.3" x2="190.5" y2="114.3" width="0.1524" layer="91"/>
+<label x="190.5" y="114.3" size="1.778" layer="95" rot="R180"/>
+</segment>
+<segment>
+<pinref part="TP12" gate="G$1" pin="1"/>
+<wire x1="137.16" y1="139.7" x2="134.62" y2="139.7" width="0.1524" layer="91"/>
+<label x="134.62" y="139.7" size="1.778" layer="95" rot="R180"/>
+</segment>
+</net>

Commit message: Updated Daughter board schematic and other boards
Parts:
- added X1: JST-XH-02-PIN-LONG-PAD, Rembrandt Electronics - JST XH Connectors v1-0:JST-XH-02-PIN-LONG-PAD
Connections:
- net GND: now also X1-2.S
- net Y_LMT: now also X1-1.S
Changed lines of the file:
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@@
 <layers>
 <layer number="1" name="Top" color="4" fill="1" visible="no" active="no"/>
+<layer number="2" name="Route2" color="1" fill="3" visible="no" active="no"/>
+<layer number="3" name="Route3" color="4" fill="3" visible="no" active="no"/>
+<layer number="4" name="Route4" color="1" fill="4" visible="no" active="no"/>
+<layer number="5" name="Route5" color="4" fill="4" visible="no" active="no"/>
+<layer number="6" name="Route6" color="1" fill="8" visible="no" active="no"/>
+<layer number="7" name="Route7" color="4" fill="8" visible="no" active="no"/>
+<layer number="8" name="Route8" color="1" fill="2" visible="no" active="no"/>
+<layer number="9" name="Route9" color="4" fill="2" visible="no" active="no"/>
+<layer number="10" name="Route10" color="1" fill="7" visible="no" active="no"/>
+<layer number="11" name="Route11" color="4" fill="7" visible="no" active="no"/>
+<layer number="12" name="Route12" color="1" fill="5" visible="no" active="no"/>
+<layer number="13" name="Route13" color="4" fill="5" visible="no" active="no"/>
+<layer number="14" name="Route14" color="1" fill="6" visible="no" active="no"/>
+<layer number="15" name="Route15" color="4" fill="6" visible="no" active="no"/>
 <layer number="16" name="Bottom" color="1" fill="1" visible="no" active="no"/>
 <layer number="17" name="Pads" color="2" fill="1" visible="no" active="no"/>
@@
 <part name="TP22" library="SparkFun-Connectors" deviceset="TEST-POINT" device="TP_15TH_THRU"/>
 <part name="U$2" library="FracktalWorks_Eagle_Library" deviceset="FRACKTALLOGO" device=""/>
+<part name="X1" library="Rembrandt Electronics - JST XH Connectors v1-0" deviceset="JST-XH-02-PIN" device="-LONG-PAD"/>
 </parts>
 <sheets>
@@
 </instance>
 <instance part="U$2" gate="G$1" x="63.5" y="2.54" smashed="yes"/>
+<instance part="X1" gate="-2" x="160.02" y="55.88" smashed="yes">
+<attribute name="NAME" x="162.56" y="55.118" size="1.524" layer="95"/>
+</instance>
+<instance part="X1" gate="-1" x="160.02" y="58.42" smashed="yes">
+<attribute name="NAME" x="162.56" y="57.658" size="1.524" layer="95"/>
+<attribute name="VALUE" x="159.258" y="59.817" size="1.778" layer="96"/>
+</instance>
 </instances>
 <busses>
@@
 <label x="134.62" y="127" size="1.778" layer="95" rot="R180"/>
 </segment>
+<segment>
+<pinref part="X1" gate="-1" pin="S"/>
+<wire x1="157.48" y1="58.42" x2="152.4" y2="58.42" width="0.1524" layer="91"/>
+<label x="152.4" y="58.42" size="1.778" layer="95"/>
+</segment>
 </net>
 <net name="GND" class="0">
@@
 <label x="86.36" y="109.22" size="1.778" layer="95" rot="R180"/>
 </segment>
-</net>
+<segment>
+<pinref part="X1" gate="-2" pin="S"/>
+<wire x1="157.48" y1="55.88" x2="152.4" y2="55.88" width="0.1524" layer="91"/>
+<label x="152.4" y="55.88" size="1.778" layer="95"/>
+</segment>
+</net>
